Commit message: + position control

File: robot.urdf (robot description, URDF)
Before this commit: robot quadrupedal_robot, 13 links, 12 joints
Links:
- link base: mass 2.792 -> 3.
- link lf_abduction_link: mass 0.0216 -> 0.25
- link lf_lower_link: mass 0.140882 -> 0.25
- link lf_upper_link: mass 0.376687 -> 0.25
- link lh_abduction_link: mass 0.0216 -> 0.25
- link lh_lower_link: mass 0.140882 -> 0.25
- link lh_upper_link: mass 0.376687 -> 0.25
- link rf_abduction_link: mass 0.0216 -> 0.25
- link rf_lower_link: mass 0.140882 -> 0.25
- link rf_upper_link: mass 0.376687 -> 0.25
- link rh_abduction_link: mass 0.0216 -> 0.25
- link rh_lower_link: mass 0.140882 -> 0.25
- link rh_upper_link: mass 0.376687 -> 0.25

Commit message: fixed inverse_kinematics with geometrical approach (TESTED)

File: robot.urdf (robot description, URDF)
Before this commit: robot quadrupedal_robot, 13 links, 12 joints
Joints:
- joint lf_abad_joint: limit lower=-2.5 upper=2.5 effort=8.0 velocity=6.0 -> lower=-3.14 upper=3.14 effort=8.0 velocity=6.0
- joint lf_hip_joint: limit lower=-2.5 upper=2.5 effort=8.0 velocity=6.0 -> lower=-3.14 upper=3.14 effort=8.0 velocity=6.0
- joint lf_knee_joint: limit lower=-2.5 upper=2.5 effort=8.0 velocity=6.0 -> lower=-3.14 upper=3.14 effort=8.0 velocity=6.0
- joint lh_abad_joint: limit lower=-2.5 upper=2.5 effort=8.0 velocity=6.0 -> lower=-3.14 upper=3.14 effort=8.0 velocity=6.0
- joint lh_hip_joint: limit lower=-2.5 upper=2.5 effort=8.0 velocity=6.0 -> lower=-3.14 upper=3.14 effort=8.0 velocity=6.0
- joint lh_knee_joint: limit lower=-2.5 upper=2.5 effort=8.0 velocity=6.0 -> lower=-3.14 upper=3.14 effort=8.0 velocity=6.0
- joint rf_abad_joint: limit lower=-2.5 upper=2.5 effort=8.0 velocity=6.0 -> lower=-3.14 upper=3.14 effort=8.0 velocity=6.0
- joint rf_hip_joint: limit lower=-2.5 upper=2.5 effort=8.0 velocity=6.0 -> lower=-3.14 upper=3.14 effort=8.0 velocity=6.0
- joint rf_knee_joint: limit lower=-2.5 upper=2.5 effort=8.0 velocity=6.0 -> lower=-3.14 upper=3.14 effort=8.0 velocity=6.0
- joint rh_abad_joint: limit lower=-2.5 upper=2.5 effort=8.0 velocity=6.0 -> lower=-3.14 upper=3.14 effort=8.0 velocity=6.0
- joint rh_hip_joint: limit lower=-2.5 upper=2.5 effort=8.0 velocity=6.0 -> lower=-3.14 upper=3.14 effort=8.0 velocity=6.0
- joint rh_knee_joint: limit lower=-2.5 upper=2.5 effort=8.0 velocity=6.0 -> lower=-3.14 upper=3.14 effort=8.0 velocity=6.0
